Commit message: Added cameraplugin for gazebo. Started work on controlling the simulated robot via Twist-messages on the cmd_vel topic

File: urdf/mikrorobot.xacro (robot description, xacro)
@@ -1,5 +1,6 @@
 <?xml version="1.0"?>
-<!-- Revolute-Revolute Manipulator -->
+<!-- Mikrorobot Mark I -->
 <robot name="mikrorobot" xmlns:xacro="http://www.ros.org/wiki/xacro">
+  <!-- rosrun gazebo_ros spawn_model -file `rospack find mikrorobot`/urdf/mikrorobot_from_xacro.urdf -urdf -z 1 -model mikrorobot -->
   <!-- Constants for robot dimensions -->
   <xacro:property name="PI" value="3.1415926535897931"/>
@@ -15,4 +16,6 @@
   <xacro:property name="wheel_offset_y" value="0.2" /> <!-- Wheel offset width-direction -->
   <xacro:property name="wheel_offset_z" value="${-height/2 + 0.05}" /> <!-- Wheel offset height-direction -->
+  <!-- Import all Gazebo-customization elements, including Gazebo colors -->
+  <xacro:include filename="$(find mikrorobot)/urdf/mikrorobot.gazebo" />
     <!-- Base Link -->
   <link name="base_link">
@@ -154,5 +157,5 @@
       <material name="black"/>
     </visual>
-        <collision>
+    <collision>
       <origin xyz="0 0 0" rpy="1.570795 0 0"/>
       <geometry>
@@ -172,5 +175,5 @@
   </link>
     <!-- Camera -->
-  <link name="camera">
+  <link name="camera_link">
     <collision>
       <origin xyz="0 0 0" rpy="0 0 0"/>
@@ -194,7 +197,7 @@
   <joint name="camera_joint" type="fixed">
     <parent link="base_link"/>
-    <child link="camera"/>
-    <origin xyz="${depth/2 - 0.05} 0 ${height/2}" rpy="-1.570795 0 -1.570795" />
-    <axis xyz="0 1 0" rpy="0 0 0" />
+    <child link="camera_link"/>
+    <origin xyz="${depth/2 - 0.03} 0 ${height/2 + 0.02}" rpy="0 0 0" />
+    <axis xyz="0 0 0" rpy="0 0 0" />
   </joint>
   <transmission name="tran_f_r">

File: urdf/mikrorobot_from_xacro.urdf (robot description, URDF)
Before this commit: robot mikrorobot, 6 links, 5 joints
Links:
- removed link camera
- added link camera_link, mass 1e-5; collision cylinder length=0.03 radius=0.02; visual cylinder length=0.03 radius=0.02
Joints:
- joint camera_joint: axis 0 1 0 -> 0 0 0; child camera -> camera_link; origin xyz=0.2 0 0.085 rpy=-1.570795 0 -1.570795 -> xyz=0.22 0 0.105 rpy=0 0 0

Commit message: added base_controller and odom

File: urdf/mikrorobot.xacro (robot description, xacro)
@@ -9,12 +9,12 @@
   <xacro:property name="width" value="0.3" />
   <xacro:property name="depth" value="0.5" />
-  <xacro:property name="height" value="0.17" />
+  <xacro:property name="height" value="0.27" />
   <xacro:property name="wheel_mass" value="1.5" />
   <xacro:property name="wheel_radius" value="0.1" />
-  <xacro:property name="wheel_width" value="0.07" />
+  <xacro:property name="wheel_width" value="0.05" />
   <xacro:property name="camera_link" value="0.05" /> <!-- Size of square 'camera' box -->
-  <xacro:property name="wheel_offset_x" value="0.2" /> <!-- Wheel offset depth-direction -->
-  <xacro:property name="wheel_offset_y" value="0.2" /> <!-- Wheel offset width-direction -->
-  <xacro:property name="wheel_offset_z" value="${-height/2 + 0.05}" /> <!-- Wheel offset height-direction -->
+  <xacro:property name="wheel_offset_x" value="0.184" /> <!-- Wheel offset depth-direction -->
+  <xacro:property name="wheel_offset_y" value="0.198" /> <!-- Wheel offset width-direction -->
+  <xacro:property name="wheel_offset_z" value="${-height/2 + 0.04}" /> <!-- Wheel offset height-direction -->
   <!-- Import all Gazebo-customization elements, including Gazebo colors -->
   <xacro:include filename="$(find mikrorobot)/urdf/mikrorobot.gazebo" />
