Commit message: Added an updatet arduinosketch Added a basic TF broadcaster. The odometry is completely missing but the rest is working fine. Added an rviz file Updated the urdf with approximate dimensions

File: urdf/mikrorobot.urdf (robot description, URDF)
Before this commit: robot mikrobot, 6 links, 5 joints
Links:
- link b_l_wheel: geometry visual cylinder length=0.015 radius=0.042
- link b_r_wheel: geometry visual cylinder length=0.015 radius=0.042
- link base_link: geometry visual box size=0.173 0.1 0.082
- link camera: geometry visual cylinder length=0.03 radius=0.02
- link f_l_wheel: geometry visual cylinder length=0.015 radius=0.042
- link f_r_wheel: geometry visual cylinder length=0.015 radius=0.042
Joints:
- joint camera_joint: origin xyz=0.4 0 0.225 rpy=0 1.570795 0 -> xyz=0.075 0 0.07 rpy=-1.570795 0 -1.570795
- joint joint_b_l_wheel: origin xyz=-0.25 0.30 0 rpy=0 0 0 -> xyz=-0.065 0.07 0 rpy=0 0 0
- joint joint_b_r_wheel: origin xyz=-0.25 -0.30 0 rpy=0 0 0 -> xyz=-0.065 -0.07 0 rpy=0 0 0
- joint joint_f_l_wheel: origin xyz=0.25 0.30 0 rpy=0 0 0 -> xyz=0.065 0.07 0 rpy=0 0 0
- joint joint_f_r_wheel: origin xyz=0.25 -0.30 0 rpy=0 0 0 -> xyz=0.065 -0.07 0 rpy=0 0 0

Commit message: Simulation now works with skid steering

File: urdf/mikrorobot.urdf (robot description, URDF)
Before this commit: robot mikrorobot, 6 links, 5 joints
Links:
- removed link b_l_wheel
- removed link b_r_wheel
- removed link camera
- removed link f_l_wheel
- removed link f_r_wheel
- added link back_left_wheel, mass 1.5; collision cylinder length=0.07 radius=0.1; visual cylinder length=0.07 radius=0.1
- added link back_right_wheel, mass 1.5; collision cylinder length=0.07 radius=0.1; visual cylinder length=0.07 radius=0.1
- added link camera_link, mass 1e-5; collision cylinder length=0.03 radius=0.02; visual cylinder length=0.03 radius=0.02
- added link front_left_wheel, mass 1.5; collision cylinder length=0.07 radius=0.1; visual cylinder length=0.07 radius=0.1
- added link front_right_wheel, mass 1.5; collision cylinder length=0.07 radius=0.1; visual cylinder length=0.07 radius=0.1
- link base_link: mass None -> 10; geometry collision box size=0.5 0.3 0.17; visual box size=0.5 0.3 0.17
Joints:
- removed joint joint_b_l_wheel
- removed joint joint_b_r_wheel
- removed joint joint_f_l_wheel
- removed joint joint_f_r_wheel
- added joint back_left_wheel_joint: type continuous, parent base_link, child back_left_wheel, origin xyz=-0.2 0.2 -0.035 rpy=0 0 0, axis 0 1 0
- added joint back_right_wheel_joint: type continuous, parent base_link, child back_right_wheel, origin xyz=-0.2 -0.2 -0.035 rpy=0 0 0, axis 0 1 0
- added joint front_left_wheel_joint: type continuous, parent base_link, child front_left_wheel, origin xyz=0.2 0.2 -0.035 rpy=0 0 0, axis 0 1 0
- added joint front_right_wheel_joint: type continuous, parent base_link, child front_right_wheel, origin xyz=0.2 -0.2 -0.035 rpy=0 0 0, axis 0 1 0
- joint camera_joint: axis 0 1 0 -> 0 0 0; child camera -> camera_link; origin xyz=0.075 0 0.07 rpy=-1.570795 0 -1.570795 -> xyz=0.22 0 0.105 rpy=0 0 0

File: urdf/mikrorobot.xacro (robot description, xacro)
@@ -45,11 +45,11 @@
   </link>
   <!-- Front Right Wheel -->
-  <joint name="joint_f_r_wheel" type="continuous">
-    <parent link="base_link"/>
-    <child link="f_r_wheel"/>
+  <joint name="front_right_wheel_joint" type="continuous">
+    <parent link="base_link"/>
+    <child link="front_right_wheel"/>
     <origin xyz="${wheel_offset_x} ${-wheel_offset_y} ${wheel_offset_z}" rpy="0 0 0" />
     <axis xyz="0 1 0" rpy="0 0 0" />
   </joint>
-  <link name="f_r_wheel">
+  <link name="front_right_wheel">
     <visual>
       <origin xyz="0 0 0" rpy="1.570795 0 0" />
@@ -79,11 +79,11 @@
   </link>
   <!-- Back Right Wheel -->
-  <joint name="joint_b_r_wheel" type="continuous">
-    <parent link="base_link"/>
-    <child link="b_r_wheel"/>
+  <joint name="back_right_wheel_joint" type="continuous">
+    <parent link="base_link"/>
+    <child link="back_right_wheel"/>
     <origin xyz="${-wheel_offset_x} ${-wheel_offset_y} ${wheel_offset_z}" rpy="0 0 0" />
     <axis xyz="0 1 0" rpy="0 0 0" />
   </joint>
-  <link name="b_r_wheel">
+  <link name="back_right_wheel">
     <visual>
       <origin xyz="0 0 0" rpy="1.570795 0 0" />
@@ -111,11 +111,11 @@
   </link>
   <!-- Front Left Wheel -->
-  <joint name="joint_f_l_wheel" type="continuous">
-    <parent link="base_link"/>
-    <child link="f_l_wheel"/>
+  <joint name="front_left_wheel_joint" type="continuous">
+    <parent link="base_link"/>
+    <child link="front_left_wheel"/>
     <origin xyz="${wheel_offset_x} ${wheel_offset_y} ${wheel_offset_z}" rpy="0 0 0" />
     <axis xyz="0 1 0" rpy="0 0 0" />
   </joint>
-  <link name="f_l_wheel">
+  <link name="front_left_wheel">
     <visual>
       <origin xyz="0 0 0" rpy="1.570795 0 0" />
@@ -143,11 +143,11 @@
   </link>
     <!-- Back Left Wheel -->
-  <joint name="joint_b_l_wheel" type="continuous">
-    <parent link="base_link"/>
-    <child link="b_l_wheel"/>
+  <joint name="back_left_wheel_joint" type="continuous">
+    <parent link="base_link"/>
+    <child link="back_left_wheel"/>
      <origin xyz="${-wheel_offset_x} ${wheel_offset_y} ${wheel_offset_z}" rpy="0 0 0" />
     <axis xyz="0 1 0" rpy="0 0 0" />
   </joint>
-  <link name="b_l_wheel">
+  <link name="back_left_wheel">
     <visual>
       <origin xyz="0 0 0" rpy="1.570795 0 0" />
@@ -203,5 +203,5 @@
   <transmission name="tran_f_r">
     <type>transmission_interface/SimpleTransmission</type>
-    <joint name="joint_f_r_wheel">
+    <joint name="front_right_wheel_joint">
       <hardwareInterface>EffortJointInterface</hardwareInterface>
     </joint>
@@ -213,5 +213,5 @@
   <transmission name="tran_b_r">
     <type>transmission_interface/SimpleTransmission</type>
-    <joint name="joint_b_r_wheel">
+    <joint name="back_right_wheel_joint">
       <hardwareInterface>EffortJointInterface</hardwareInterface>
     </joint>
@@ -223,5 +223,5 @@
   <transmission name="tran_f_l">
     <type>transmission_interface/SimpleTransmission</type>
-    <joint name="joint_f_l_wheel">
+    <joint name="front_left_wheel_joint">
       <hardwareInterface>EffortJointInterface</hardwareInterface>
     </joint>
@@ -233,5 +233,5 @@
   <transmission name="tran_b_l">
     <type>transmission_interface/SimpleTransmission</type>
-    <joint name="joint_b_l_wheel">
+    <joint name="back_left_wheel_joint">
       <hardwareInterface>EffortJointInterface</hardwareInterface>
     </joint>

Commit message: Added lidar to gazebo model

File: urdf/mikrorobot.urdf (robot description, URDF)
Before this commit: robot mikrorobot, 6 links, 5 joints
Links:
- added link laser_link, mass 1e-5; collision cylinder length=0.03 radius=0.02; visual cylinder length=0.03 radius=0.02
Joints:
- added joint laser_joint: type fixed, parent base_link, child laser_link, origin xyz=0 0 0.105 rpy=0 0 0, axis 0 0 0

File: urdf/mikrorobot.xacro (robot description, xacro)
@@ -201,4 +201,32 @@
     <axis xyz="0 0 0" rpy="0 0 0" />
   </joint>
+      <!-- Laser -->
+  <link name="laser_link">
+    <collision>
+      <origin xyz="0 0 0" rpy="0 0 0"/>
+      <geometry>
+	<cylinder length="0.03" radius ="0.02"/>
+      </geometry>
+    </collision>
+    <visual>
+      <origin xyz="0 0 0" rpy="0 0 0" />
+      <geometry>
+          <cylinder length="0.03" radius="0.02" />
+      </geometry>
+      <material name="black"/>
+    </visual>
+    <inertial>
+      <mass value="1e-5" />
+      <origin xyz="0 0 0" rpy="0 0 0"/>
+      <inertia ixx="1e-6" ixy="0" ixz="0" iyy="1e-6" iyz="0" izz="1e-6" />
+    </inertial>
+  </link>
+  <joint name="laser_joint" type="fixed">
+    <parent link="base_link"/>
+    <child link="laser_link"/>
+    <origin xyz="0 0 ${height/2 + 0.02}" rpy="0 0 0" />
+    <axis xyz="0 0 0" rpy="0 0 0" />
+  </joint>
+  <!-- Transmissions -->
   <transmission name="tran_f_r">
     <type>transmission_interface/SimpleTransmission</type>

Commit message: Broke odometry while trying to fix it. Making progress

File: urdf/mikrorobot.urdf (robot description, URDF)
Before this commit: robot mikrorobot, 7 links, 6 joints
Links:
- added link base_footprint; visual box size=0.001 0.001 0.001
Joints:
- added joint base_link_joint: type fixed, parent base_footprint, child base_link, origin xyz=0.0 0 0.085 rpy=0 0 0

File: urdf/mikrorobot.xacro (robot description, xacro)
@@ -1,5 +1,5 @@
 <?xml version="1.0"?>
 <!-- Mikrorobot Mark I -->
-<robot name="mikrorobot" xmlns:xacro="http://www.ros.org/wiki/xacro">
+<robot name="mikrorobot" xmlns:xacro="http://www.roxs.org/wiki/xacro">
   <!-- Use this command to spawn the model in gazebo: rosrun gazebo_ros spawn_model -file `rospack find mikrorobot`/urdf/mikrorobot.urdf -urdf -z 1 -model mikrorobot -->
   <!-- Use this command to generate the urdf (use two -'s in front of inorder): rosrun xacro xacro -inorder mikrorobot.xacro > mikrorobot.urdf -->
@@ -19,4 +19,18 @@
   <!-- Import all Gazebo-customization elements, including Gazebo colors -->
   <xacro:include filename="$(find mikrorobot)/urdf/mikrorobot.gazebo" />
+  <!-- root link, on the ground just below the model origin -->
+  <link name="base_footprint">
+   <visual>
+      <origin xyz="0 0 0" rpy="0 0 0" />
+      <geometry>
+        <box size="0.001 0.001 0.001" />
+      </geometry>
+    </visual>
+  </link>
+  <joint name="base_link_joint" type="fixed">
+    <origin xyz="0.0 0 ${height/2}" rpy="0 0 0" />
+    <parent link="base_footprint"/>
+    <child link="base_link" />
+  </joint>
     <!-- Base Link -->
   <link name="base_link">

Commit message: fixed pid-controller issue, done some work towards launchfiles being usable on the completed robot

File: urdf/mikrorobot.urdf (robot description, URDF)
Before this commit: robot mikrorobot, 7 links, 6 joints
Links:
- removed link laser_link
- added link laser_frame, mass 1e-5; collision cylinder length=0.03 radius=0.02; visual cylinder length=0.03 radius=0.02
- link back_left_wheel: geometry collision cylinder length=0.05 radius=0.1; visual cylinder length=0.05 radius=0.1
- link back_right_wheel: geometry collision cylinder length=0.05 radius=0.1; visual cylinder length=0.05 radius=0.1
- link base_link: geometry collision box size=0.5 0.3 0.27; visual box size=0.5 0.3 0.27
- link front_left_wheel: geometry collision cylinder length=0.05 radius=0.1; visual cylinder length=0.05 radius=0.1
- link front_right_wheel: geometry collision cylinder length=0.05 radius=0.1; visual cylinder length=0.05 radius=0.1
Joints:
- joint back_left_wheel_joint: origin xyz=-0.2 0.2 -0.035 rpy=0 0 0 -> xyz=-0.184 0.198 -0.095 rpy=0 0 0
- joint back_right_wheel_joint: origin xyz=-0.2 -0.2 -0.035 rpy=0 0 0 -> xyz=-0.184 -0.198 -0.095 rpy=0 0 0
- joint camera_joint: origin xyz=0.22 0 0.105 rpy=0 0 0 -> xyz=0.22 0 0.155 rpy=0 0 0
- joint front_left_wheel_joint: origin xyz=0.2 0.2 -0.035 rpy=0 0 0 -> xyz=0.184 0.198 -0.095 rpy=0 0 0
- joint front_right_wheel_joint: origin xyz=0.2 -0.2 -0.035 rpy=0 0 0 -> xyz=0.184 -0.198 -0.095 rpy=0 0 0
- joint laser_joint: child laser_link -> laser_frame; origin xyz=0 0 0.105 rpy=0 0 0 -> xyz=0 0 0.155 rpy=0 0 0

File: urdf/mikrorobot.xacro (robot description, xacro)
@@ -203,5 +203,5 @@
   </joint>
       <!-- Laser -->
-  <link name="laser_link">
+  <link name="laser_frame">
     <collision>
       <origin xyz="0 0 0" rpy="0 0 0"/>
@@ -225,5 +225,5 @@
   <joint name="laser_joint" type="fixed">
     <parent link="base_link"/>
-    <child link="laser_link"/>
+    <child link="laser_frame"/>
     <origin xyz="0 0 ${height/2 + 0.02}" rpy="0 0 0" />
     <axis xyz="0 0 0" rpy="0 0 0" />

Commit message: fikset så laser_frame er sånn nogenlunde riktig, må måles opp. Driver å tweaker på odometrien, men det er fortsatt noe galt med vinkelmålingene

File: urdf/mikrorobot.urdf (robot description, URDF)
Before this commit: robot mikrorobot, 7 links, 6 joints
Joints:
- joint laser_joint: origin xyz=0 0 0.155 rpy=0 0 0 -> xyz=0.2 0 0.255 rpy=0 0 3.14159265359

File: urdf/mikrorobot.xacro (robot description, xacro)
@@ -226,5 +226,5 @@
     <parent link="base_link"/>
     <child link="laser_frame"/>
-    <origin xyz="0 0 ${height/2 + 0.02}" rpy="0 0 0" />
+    <origin xyz="${depth/2 - 0.05} 0 ${height/2 + 0.12}" rpy="0 0 ${PI}" />
     <axis xyz="0 0 0" rpy="0 0 0" />
   </joint>

Commit message: Fikset kommunikasjon med to Rpis

File: urdf/mikrorobot.urdf (robot description, URDF)
Before this commit: robot mikrorobot, 7 links, 6 joints
Links:
- added link imu_frame, mass 1e-5
Joints:
- added joint imu_joint: type fixed, parent base_link, child imu_frame, origin xyz=0.15 -0.02 0.265 rpy=0 3.14159265359 0, axis 0 0 0

File: urdf/mikrorobot.xacro (robot description, xacro)
@@ -229,4 +229,18 @@
     <axis xyz="0 0 0" rpy="0 0 0" />
   </joint>
+        <!-- IMU -->
+  <link name="imu_frame">
+    <inertial>
+      <mass value="1e-5" />
+      <origin xyz="0 0 0" rpy="0 0 0"/>
+      <inertia ixx="1e-6" ixy="0" ixz="0" iyy="1e-6" iyz="0" izz="1e-6" />
+    </inertial>
+  </link>
+  <joint name="imu_joint" type="fixed">
+    <parent link="base_link"/>
+    <child link="imu_frame"/>
+    <origin xyz="${depth/2 - 0.10} ${-0.02} ${- height/2 + 0.4}" rpy="0 ${PI} 0" />
+    <axis xyz="0 0 0" rpy="0 0 0" />
+  </joint>
   <!-- Transmissions -->
   <transmission name="tran_f_r">

Commit message: Fikset navigasjonsstacken, må tunes masse, men VIRKER :D

File: urdf/mikrorobot.urdf (robot description, URDF)
Before this commit: robot mikrorobot, 8 links, 7 joints
Joints:
- joint imu_joint: origin xyz=0.15 -0.02 0.265 rpy=0 3.14159265359 0 -> xyz=0.15 -0.02 0.265 rpy=0.785398163397 3.14159265359 0

File: urdf/mikrorobot.xacro (robot description, xacro)
@@ -240,5 +240,5 @@
     <parent link="base_link"/>
     <child link="imu_frame"/>
-    <origin xyz="${depth/2 - 0.10} ${-0.02} ${- height/2 + 0.4}" rpy="0 ${PI} 0" />
+    <origin xyz="${depth/2 - 0.10} ${-0.02} ${- height/2 + 0.4}" rpy="${PI/4} ${PI} 0" />
     <axis xyz="0 0 0" rpy="0 0 0" />
   </joint>

Commit message: Lagt til støtte for structure i urdf

File: urdf/mikrorobot.urdf (robot description, URDF)
Before this commit: robot mikrorobot, 8 links, 7 joints
Links:
- added link camera_depth_optical_frame, mass 1e-5; collision cylinder length=0.03 radius=0.02; visual cylinder length=0.03 radius=0.02
Joints:
- added joint structure_camera_joint: type fixed, parent base_link, child camera_depth_optical_frame, origin xyz=0.28 0 0.135 rpy=-1.57079632679 0 -1.57079632679, axis 0 0 0

File: urdf/mikrorobot.xacro (robot description, xacro)
@@ -202,4 +202,31 @@
     <axis xyz="0 0 0" rpy="0 0 0" />
   </joint>
+      <!-- Structure Camera -->
+  <link name="camera_depth_optical_frame">
+    <collision>
+      <origin xyz="0 0 0" rpy="0 0 0"/>
+      <geometry>
+	<cylinder length="0.03" radius ="0.02"/>
+      </geometry>
+    </collision>
+    <visual>
+      <origin xyz="0 0 0" rpy="0 0 0" />
+      <geometry>
+          <cylinder length="0.03" radius="0.02" />
+      </geometry>
+      <material name="black"/>
+    </visual>
+    <inertial>
+      <mass value="1e-5" />
+      <origin xyz="0 0 0" rpy="0 0 0"/>
+      <inertia ixx="1e-6" ixy="0" ixz="0" iyy="1e-6" iyz="0" izz="1e-6" />
+    </inertial>
+  </link>
+  <joint name="structure_camera_joint" type="fixed">
+    <parent link="base_link"/>
+    <child link="camera_depth_optical_frame"/>
+    <origin xyz="${depth/2 + 0.03} 0 ${height/2}" rpy="${-PI/2} 0 ${-PI/2}" />
+    <axis xyz="0 0 0" rpy="0 0 0" />
+  </joint>
       <!-- Laser -->
   <link name="laser_frame">
